Commit message: adding the navigation stack

File: r2d2_description/urdf/r2d2.gazebo.xacro (robot description, xacro)
@@ -23,7 +23,7 @@
 			<torque>20</torque>
 			<broadcastTF>1</broadcastTF>
-			<odometryFrame>map</odometryFrame>
+			<odometryFrame>odom</odometryFrame>
 			<commandTopic>cmd_vel</commandTopic>
-			<odometryTopic>r2d2/odom</odometryTopic>
+			<odometryTopic>/odom</odometryTopic>
 			<robotBaseFrame>base_link</robotBaseFrame>
 		</plugin>
@@ -60,5 +60,5 @@
 			</ray>
 			<plugin name="gazebo_ros_head_hokuyo_controller" filename="libgazebo_ros_gpu_laser.so">
-				<topicName>/r2d2/laser/scan</topicName>
+				<topicName>/scan</topicName>
 				<frameName>hokuyo_link</frameName>
 			</plugin>

File: r2d2_description/urdf/r2d2.urdf.xacro (robot description, xacro)
@@ -5,10 +5,5 @@
  	-->
 	<xacro:include filename="$(find r2d2_description)/urdf/r2d2.structure.xacro" />
-	<link name="base_footprint" />
 	<link name="base_link" />
-	<joint name="base_footprint_base_link_joint" type="fixed">
-		<parent link="base_footprint"/>
-		<child link="base_link"/>
-	</joint>
 	<xacro:r2d2_structure name="r2d2_structure" parent_link="base_link"/>
 </robot>
