Commit message: improvements in the robot model

File: r2d2_description/urdf/r2d2.gripper.xacro (robot description, xacro)
@@ -22,5 +22,5 @@
 			<parent link="${parent_link}"/>
 			<child link="gripper_pole"/>
-			<limit effort="1000.0" lower="-${torsowidth*2-.02}" upper="0" velocity="0.5"/>
+			<limit effort="1000.0" lower="-${torsowidth*2-.02}" upper="-0.1" velocity="0.5"/>
 			<origin rpy="0 0 0" xyz="${torsowidth-.01} 0 .2"/>
 			<limit effort="30" velocity="0.2"/>

File: r2d2_description/urdf/r2d2.leg.xacro (robot description, xacro)
@@ -16,5 +16,5 @@
 				<origin xyz="0 0 -${leglen/2}" rpy="0 ${pi/2} 0"/>
 			</collision>
-			<xacro:default_inertial mass="10"/>
+			<xacro:default_inertial mass="2"/>
 		</link>
 		<xacro:gazebo_material link="${prefix}_leg" color="White"/>
@@ -31,5 +31,5 @@
 				</geometry>
 			</collision>
-			<xacro:default_inertial mass="10"/>
+			<xacro:default_inertial mass="20"/>
 		</link>
 		<xacro:gazebo_material link="${prefix}_leg_base" color="White"/>

File: r2d2_description/urdf/r2d2.wheel.xacro (robot description, xacro)
@@ -18,5 +18,5 @@
 				<origin xyz="0 0 0" rpy="0 0 0" />
 			</collision>
-			<xacro:default_inertial mass="1"/>
+			<xacro:default_inertial mass="2"/>
 		</link>
 		<xacro:gazebo_material link="${prefix}_${suffix}_wheel" color="Black"/>
